Commit message: refactor: remove Kalman prediction (direct q_safe passthrough); fix RViz passive joints via URDF mimic tags; remove jsp_gui from display.launch

File: src/mg400_description/urdf/mg400.xacro (robot description, xacro)
@@ -479,4 +479,6 @@
           effort="0"
           velocity="0" />
+      <!-- Passive: mirrors j2_1 to form the parallel 4-bar linkage -->
+      <mimic joint="${prefix}mg400_j2_1" multiplier="1" offset="0" />
     </joint>
     <joint
@@ -494,4 +496,6 @@
           effort="0"
           velocity="0" />
+      <!-- Passive: negative of j2_1 to keep bottom rods parallel -->
+      <mimic joint="${prefix}mg400_j2_1" multiplier="-1" offset="0" />
     </joint>
     <joint
@@ -509,4 +513,6 @@
           effort="0"
           velocity="0" />
+      <!-- Passive: negative of j2_1 (via j2_2 mirror) -->
+      <mimic joint="${prefix}mg400_j2_1" multiplier="-1" offset="0" />
     </joint>
     <joint
@@ -524,4 +530,6 @@
           effort="0"
           velocity="0" />
+      <!-- Passive: negative of j3 to enforce end-effector perpendicularity -->
+      <mimic joint="${prefix}mg400_j3" multiplier="-1" offset="0" />
     </joint>
     <joint
@@ -539,4 +547,6 @@
           effort="0"
           velocity="0" />
+      <!-- Passive: mirrors j3 -->
+      <mimic joint="${prefix}mg400_j3" multiplier="1" offset="0" />
     </joint>
     <joint

Commit message: fix: restore original RViz mimic joints and synchronous command sending to stop oscillation

File: src/mg400_description/urdf/mg400.xacro (robot description, xacro)
@@ -1,9 +1,7 @@
 <?xml version="1.0" encoding="UTF-8"?>
 <robot xmlns:xacro="http://ros.org/wiki/xacro">
-  <!-- constants -->
   <xacro:include
       filename="$(find mg400_description)/urdf/common/constants.xacro"
       ns="const" />
-  <!-- Base path for meshes -->
   <xacro:property
       name="BASE_PATH"
@@ -51,5 +49,4 @@
       <color rgba="0.2 0.0 0.0 0.5" />
     </material>
-    <!-- links -->
     <link name="${prefix}mg400_base_link">
       <inertial>
@@ -300,4 +297,11 @@
         </geometry>
       </collision>
+    </link>
+    <link name="${prefix}fake_link">
+       <inertial>
+        <origin xyz="0 0 0" rpy="0 0 0" />
+        <mass value="0.001" />
+        <inertia ixx="0.0001" ixy="0" ixz="0" iyy="0.0001" iyz="0" izz="0.0001" />
+      </inertial>
     </link>
     <link name="${prefix}mg400_link4_3">
@@ -407,5 +411,4 @@
       </link>
     </xacro:if>
-    <!-- joints -->
     <joint
         name="${prefix}mg400_base_joint"
@@ -479,23 +482,5 @@
           effort="0"
           velocity="0" />
-      <!-- Passive: mirrors j2_1 to form the parallel 4-bar linkage -->
-      <mimic joint="${prefix}mg400_j2_1" multiplier="1" offset="0" />
-    </joint>
-    <joint
-        name="${prefix}mg400_j3_1"
-        type="revolute">
-      <origin
-          xyz="-0.0010512570171516 0.0357748756218898 0.175001164344716"
-          rpy="0 0 0" />
-      <parent link="${prefix}mg400_link2_1" />
-      <child link="${prefix}mg400_link3_1" />
-      <axis xyz="0 1 0" />
-      <limit
-          lower="-3.14"
-          upper="3.14"
-          effort="0"
-          velocity="0" />
-      <!-- Passive: negative of j2_1 to keep bottom rods parallel -->
-      <mimic joint="${prefix}mg400_j2_1" multiplier="-1" offset="0" />
+      <mimic joint="${prefix}mg400_j2_1" />
     </joint>
     <joint
@@ -513,6 +498,52 @@
           effort="0"
           velocity="0" />
-      <!-- Passive: negative of j2_1 (via j2_2 mirror) -->
-      <mimic joint="${prefix}mg400_j2_1" multiplier="-1" offset="0" />
+      <mimic joint="${prefix}mg400_j2_2" multiplier="-1" />
+    </joint>
+    <joint
+        name="${prefix}mg400_j3"
+        type="revolute">
+      <origin
+          xyz="-0.0010512570171516 0.0357748756218898 0.175001164344716"
+          rpy="0 0 0" />
+      <parent link="${prefix}mg400_link2_1" />
+      <child link="${prefix}fake_link" />
+      <axis xyz="0 1 0" />
+      <limit
+          lower="-3.14"
+          upper="3.14"
+          effort="0"
+          velocity="0" />
+    </joint>
+    <joint
+        name="${prefix}mg400_j3_1"
+        type="revolute">
+      <origin
+          xyz="0 0 0"
+          rpy="0 0 0" />
+      <parent link="${prefix}fake_link" />
+      <child link="${prefix}mg400_link3_1" />
+      <axis xyz="0 1 0" />
+      <limit
+          lower="-3.14"
+          upper="3.14"
+          effort="0"
+          velocity="0" />
+      <mimic joint="${prefix}mg400_j3_2" />
+    </joint>
+    <joint
+        name="${prefix}mg400_j4_2"
+        type="revolute">
+      <origin
+          xyz="0.0679 0.0005 0.011972"
+          rpy="0 0 0" />
+      <parent link="${prefix}mg400_link3_2" />
+      <child link="${prefix}mg400_link4_2" />
+      <axis xyz="0 1 0" />
+      <limit
+          lower="-3.14"
+          upper="3.14"
+          effort="0"
+          velocity="0" />
+      <mimic joint="${prefix}mg400_j3" />
     </joint>
     <joint
@@ -530,23 +561,5 @@
           effort="0"
           velocity="0" />
-      <!-- Passive: negative of j3 to enforce end-effector perpendicularity -->
-      <mimic joint="${prefix}mg400_j3" multiplier="-1" offset="0" />
-    </joint>
-    <joint
-        name="${prefix}mg400_j4_2"
-        type="revolute">
-      <origin
-          xyz="0.0679 0.0005 0.011972"
-          rpy="0 0 0" />
-      <parent link="${prefix}mg400_link3_2" />
-      <child link="${prefix}mg400_link4_2" />
-      <axis xyz="0 1 0" />
-      <limit
-          lower="-3.14"
-          upper="3.14"
-          effort="0"
-          velocity="0" />
-      <!-- Passive: mirrors j3 -->
-      <mimic joint="${prefix}mg400_j3" multiplier="1" offset="0" />
+      <mimic joint="${prefix}mg400_j4_2" multiplier="-1" />
     </joint>
     <joint
